Commit message: Update Car to be diff. move

File: src/amr_description/urdf/amr_base.xacro (robot description, xacro)
@@ -1,4 +1,5 @@
 <?xml version="1.0"?>
 <robot xmlns:xacro="http://www.ros.org/wiki/xacro" name="amr_robot">
+    <xacro:include filename="inertial_macros.xacro" />
     <xacro:property name="chassis_length" value="0.4"/>
     <xacro:property name="chassis_width" value="0.3"/>
@@ -9,11 +10,13 @@
     <link name="chassis">
         <visual>
-            <geometry>
-                <box size="${chassis_length} ${chassis_width} ${chassis_height}"/>
-            </geometry>
-            <material name="blue">
-                <color rgba="0.0 0.0 0.8 1.0"/>
-            </material>
+            <geometry><box size="${chassis_length} ${chassis_width} ${chassis_height}"/></geometry>
+            <material name="blue"><color rgba="0.0 0.0 0.8 1.0"/></material>
         </visual>
+        <collision>
+            <geometry><box size="${chassis_length} ${chassis_width} ${chassis_height}"/></geometry>
+        </collision>
+        <xacro:inertial_box mass="5.0" x="${chassis_length}" y="${chassis_width}" z="${chassis_height}">
+            <origin xyz="0 0 0" rpy="0 0 0"/>
+        </xacro:inertial_box>
     </link>
     <joint name="base_to_chassis" type="fixed">
@@ -22,25 +25,62 @@
         <origin xyz="0 0 0.05" rpy="0 0 0"/>
     </joint>
-    <xacro:macro name="wheel" params="prefix x_reflect y_reflect">
+    <xacro:macro name="wheel" params="prefix y_reflect">
         <link name="${prefix}_wheel">
             <visual>
                 <origin xyz="0 0 0" rpy="${pi/2} 0 0"/>
-                <geometry>
-                    <cylinder radius="${wheel_radius}" length="${wheel_thickness}"/>
-                </geometry>
-                <material name="black">
-                    <color rgba="0.1 0.1 0.1 1.0"/>
-                </material>
+                <geometry><cylinder radius="${wheel_radius}" length="${wheel_thickness}"/></geometry>
+                <material name="black"><color rgba="0.1 0.1 0.1 1.0"/></material>
             </visual>
+            <collision>
+                <origin xyz="0 0 0" rpy="${pi/2} 0 0"/>
+                <geometry><cylinder radius="${wheel_radius}" length="${wheel_thickness}"/></geometry>
+            </collision>
+            <xacro:inertial_cylinder mass="0.5" length="${wheel_thickness}" radius="${wheel_radius}">
+                <origin xyz="0 0 0" rpy="${pi/2} 0 0"/>
+            </xacro:inertial_cylinder>
         </link>
         <joint name="${prefix}_wheel_joint" type="continuous">
             <parent link="chassis"/>
             <child link="${prefix}_wheel"/>
-            <origin xyz="${x_reflect * (chassis_length/2 - 0.05)} ${y_reflect * (chassis_width/2 + wheel_thickness/2)} -0.02" rpy="0 0 0"/>
-            <axis xyz="0 1 0"/> </joint>
+            <origin xyz="0 ${y_reflect * (chassis_width/2 + wheel_thickness/2)} -0.02" rpy="0 0 0"/>
+            <axis xyz="0 1 0"/>
+        </joint>
     </xacro:macro>
-    <xacro:wheel prefix="front_left" x_reflect="1" y_reflect="1" />
-    <xacro:wheel prefix="front_right" x_reflect="1" y_reflect="-1" />
-    <xacro:wheel prefix="rear_left" x_reflect="-1" y_reflect="1" />
-    <xacro:wheel prefix="rear_right" x_reflect="-1" y_reflect="-1" />
+    <xacro:wheel prefix="left" y_reflect="1" />
+    <xacro:wheel prefix="right" y_reflect="-1" />
+    <xacro:macro name="caster_wheel" params="prefix x_offset">
+        <link name="${prefix}_caster">
+            <visual>
+                <geometry><sphere radius="0.03"/></geometry>
+                <material name="black"/>
+            </visual>
+            <collision>
+                <geometry><sphere radius="0.03"/></geometry>
+            </collision>
+            <xacro:inertial_box mass="0.1" x="0.06" y="0.06" z="0.06">
+                <origin xyz="0 0 0" rpy="0 0 0"/>
+            </xacro:inertial_box>
+        </link>
+        <gazebo reference="${prefix}_caster">
+            <mu1>0.001</mu1>
+            <mu2>0.001</mu2>
+        </gazebo>
+        <joint name="${prefix}_caster_joint" type="fixed">
+            <parent link="chassis"/>
+            <child link="${prefix}_caster"/>
+            <origin xyz="${x_offset} 0 -0.04" rpy="0 0 0"/>
+        </joint>
+    </xacro:macro>
+    <xacro:caster_wheel prefix="front" x_offset="0.15" />
+    <xacro:caster_wheel prefix="rear" x_offset="-0.15" />
+    <gazebo>
+        <plugin filename="gz-sim-diff-drive-system" name="gz::sim::systems::DiffDrive">
+            <left_joint>left_wheel_joint</left_joint>
+            <right_joint>right_wheel_joint</right_joint>
+            <wheel_separation>0.34</wheel_separation>
+            <wheel_radius>0.05</wheel_radius>
+            <odom_publish_frequency>30</odom_publish_frequency>
+            <topic>cmd_vel</topic>
+        </plugin>
+    </gazebo>
 </robot>
